File: pa_usrp_ui.kicad_pcb (KiCad board)
At the start: 4 copper layers, 59 x 39 mm, 18 parts, among them J1 BWSMA-KE-P001, J2 BWSMA-KE-P001, J3 2118722-2, U1 QPA9418TR13

Commit message: Adding lna uplink
Parts:
- removed C10, C3, C9: 0.1uF, Capacitor_SMD:C_0603_1608Metric
- removed C2, C6: 10.0uF, Diode_SMD:D_0603_1608Metric
- removed C4, C7: 1000pF, Capacitor_SMD:C_0603_1608Metric
- removed C8: 100pF, Capacitor_SMD:C_0603_1608Metric
- removed R1: 0, Resistor_SMD:R_0603_1608Metric
- removed U1: QPA9418TR13, fooptrints:DFN-14_L7.0-W7.0-P1.06-TL-EP_QPA9418TR13
- added C1: 100pF, Capacitor_SMD:C_0603_1608Metric, F.Cu at (129.0, 89.5)
- added C11: 100pF, Capacitor_SMD:C_0603_1608Metric, F.Cu at (140.5, 87.0)
- added C12: 100pF, Capacitor_SMD:C_0603_1608Metric, F.Cu at (134.5, 86.0)
- added C5: 100pF, Capacitor_SMD:C_0603_1608Metric, F.Cu at (140.5, 90.5)
- added J4: Conn_01x03_Pin, Connector_PinHeader_2.54mm:PinHeader_1x03_P2.54mm_Vertical, F.Cu at (142.0, 105.2)
- added J5: HX DC002-1.3, fooptrints:DC-IN-TH_HANXIA_HX-DC002-1.3, F.Cu at (119.0, 105.3)
- added L1: 18nH, Inductor_SMD:L_0603_1608Metric, F.Cu at (137.2, 88.7)
- added R3: 10k, Resistor_SMD:R_0603_1608Metric, F.Cu at (135.5, 94.0)
- added R4: 33k, Resistor_SMD:R_0603_1608Metric, F.Cu at (133.5, 101.5)
- added U2: TQP3M9036, fooptrints:DFN-8_L2.0-W2.0-P0.50-BL-EP, F.Cu at (133.1, 89.8)
- TP1: value VCC1 -> GND
- TP2: value VCC2 -> SHDIN
- moved TP3 36.9 mm to (125.5, 105.5)
- moved TP2 32.2 mm to (130.5, 105.5), turned to 0 degrees
- moved R2 7.55 mm to (144.0, 86.2), turned to -90 degrees
- moved F1 1.12 mm to (145.2, 89.5)
- moved TP1 1.12 mm to (135.5, 105.5), turned to 0 degrees
- moved J1 1.08 mm to (104.5, 89.5)
- moved J3 1.07 mm to (131.0, 86.4)
- moved J2 1.02 mm to (158.5, 89.5)
Connections:
- R2 pad 2: Net-(F1-B3UL) -> Net-(F1-B3DL)
- TP1 pad 1: VCC2 -> GNDREF
- TP2 pad 1: VCC1 -> /SHDIN
- TP3 pad 1: VREF -> VDD
Routing:
- net /SHDIN: track 0.00 -> 16.8 mm
- net GNDREF: track 77.2 -> 61.5 mm, vias 117 -> 38
- net VDD: track 0.00 -> 12.4 mm, vias 0 -> 8
- net Net-(U2-Shutdown): track 0.00 -> 12.4 mm
- net Net-(U1-VREF): track 9.81 -> 0.00 mm, vias 4 -> 0
- net Net-(F1-B3DL): track 10.6 -> 1.76 mm
- net VCC2: track 6.26 -> 0.00 mm, vias 4 -> 0
- net Net-(U2-RFout): track 0.00 -> 6.10 mm
- net VCC1: track 4.47 -> 0.00 mm, vias 4 -> 0
- net Net-(U2-RFin): track 0.00 -> 2.37 mm
- net Net-(F1-B3UL): track 2.05 -> 3.25 mm
- net Net-(C1-Pad1): track 23.6 -> 22.4 mm
- net VREF: track 1.07 -> 0.00 mm, vias 1 -> 0
- added copper zone on In1.Cu, net GNDREF
- added copper zone on In2.Cu, net VDD
- removed copper zone on B.Cu, net GNDREF
- removed copper zone on F.Cu, net GNDREF
- removed copper zone on F.Cu, net VCC1
- removed copper zone on F.Cu, net VCC2
- removed copper zone on F.Cu, net VREF
Other:
- board text added: "5V"
- board text added: "GND"
- board text added: "LNA"
- board text added: "S/N: LNAIGW001170926"
- board text added: "SHDIN"
- board text removed: "S/N: PAUIGW001170926"

Commit message: adding ngwe
Parts:
- removed C1, C11, C5: 100pF, Capacitor_SMD:C_0603_1608Metric
- added C13: 100pF, Capacitor_SMD:C_0402_1005Metric, F.Cu at (134.5, 84.0)
- added C14: 100pF, Capacitor_SMD:C_0402_1005Metric, F.Cu at (140.5, 90.5)
- added C15: 100pF, Capacitor_SMD:C_0402_1005Metric, F.Cu at (129.0, 89.5)
- C12: value 100pF -> 1uF; footprint Capacitor_SMD:C_0603_1608Metric -> Capacitor_SMD:C_0402_1005Metric
- L1: value 18nH -> 68nH
Routing:
- net VDD: track 12.4 -> 16.0 mm, vias 8 -> 9
- net GNDREF: track 61.5 -> 64.4 mm, vias 38 -> 70

Commit message: add lna downlink
Parts:
- moved R2 6.84 mm to (144.5, 93.0), turned to 90 degrees
- moved C14 2.06 mm to (141.0, 88.5)
Connections:
- C14 pad 2: Net-(F1-B3UL) -> Net-(F1-B3DL)
- R2 pad 2: Net-(F1-B3DL) -> Net-(F1-B3UL)
Routing:
- net VDD: track 16.0 -> 13.9 mm, vias 9 -> 7
- net Net-(F1-B3UL): track 3.25 -> 1.77 mm
- net Net-(F1-B3DL): track 1.76 -> 3.08 mm
- net GNDREF: track 64.4 -> 63.7 mm, vias 70 -> 71
Changed lines of the file:
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@@
 	(footprint "Capacitor_SMD:C_0402_1005Metric"
 		(layer "F.Cu")
-		(at 140.5 90.5)
+		(at 141 88.5)
 		(descr "Capacitor SMD 0402 (1005 Metric), square (rectangular) end terminal, IPC-7351 nominal, (Body size source: IPC-SM-782 page 76, https://www.pcb-3d.com/wordpress/wp-content/uploads/ipc-sm-782a_amendment_1_and_2.pdf)")
 		(tags "capacitor")
@@
 			(layers "F.Cu" "F.Mask" "F.Paste")
 			(roundrect_rratio 0.25)
-			(net "Net-(F1-B3UL)")
+			(net "Net-(F1-B3DL)")
 			(pintype "passive")
 		)
@@
 	(footprint "Resistor_SMD:R_0603_1608Metric"
 		(layer "F.Cu")
-		(at 144 86.175 -90)
+		(at 144.5 93 90)
 		(descr "Resistor SMD 0603 (1608 Metric), square (rectangular) end terminal, IPC-7351 nominal, (Body size source: IPC-SM-782 page 72, https://www.pcb-3d.com/wordpress/wp-content/uploads/ipc-sm-782a_amendment_1_and_2.pdf)")
 		(tags "resistor")
@@
 		)
 		(property "lcsc_id" "C849792"
-			(at 0 0 270)
+			(at 0 0 90)
 			(unlocked yes)
 			(layer "F.Fab")
@@
 		)
 		(property "price" "0.0263"
-			(at 0 0 270)
+			(at 0 0 90)
 			(unlocked yes)
 			(layer "F.Fab")
@@
 		(duplicate_pad_numbers_are_jumpers no)
 		(fp_line
-			(start -0.237258 0.5225)
-			(end 0.237258 0.5225)
+			(start -0.237258 -0.5225)
+			(end 0.237258 -0.5225)
 			(stroke
 				(width 0.12)
@@
 		)
 		(fp_line
-			(start -0.237258 -0.5225)
-			(end 0.237258 -0.5225)
+			(start -0.237258 0.5225)
+			(end 0.237258 0.5225)
 			(stroke
 				(width 0.12)
@@
 		)
 		(pad "1" smd roundrect
-			(at -0.825 0 270)
+			(at -0.825 0 90)
 			(size 0.8 0.95)
 			(layers "F.Cu" "F.Mask" "F.Paste")
@@
 		)
 		(pad "2" smd roundrect
-			(at 0.825 0 270)
+			(at 0.825 0 90)
 			(size 0.8 0.95)
 			(layers "F.Cu" "F.Mask" "F.Paste")
 			(roundrect_rratio 0.25)
-			(net "Net-(F1-B3DL)")
+			(net "Net-(F1-B3UL)")
 			(pintype "passive")
 		)
@@
 	)
 	(segment
-		(start 139.5 87)
-		(end 139.725 87)
-		(width 0.45)
-		(layer "F.Cu")
-		(net "VDD")
-	)
-	(segment
 		(start 124.5 106.5)
 		(end 123.5 106.5)
@@
 	)
 	(segment
-		(start 139.725 86.225)
-		(end 139.5 86)
-		(width 0.45)
-		(layer "F.Cu")
-		(net "VDD")
-	)
-	(segment
 		(start 126 105)
 		(end 124.5 106.5)
@@
 	)
 	(segment
-		(start 139 87.5)
-		(end 139.5 87)
-		(width 0.45)
-		(layer "F.Cu")
-		(net "VDD")
-	)
-	(segment
-		(start 139.725 87)
-		(end 139.725 86.225)
-		(width 0.45)
-		(layer "F.Cu")
-		(net "VDD")
-	)
-	(segment
 		(start 138 87)
 		(end 137.187395 87.812605)
@@
 	)
 	(via
-		(at 139.5 86)
-		(size 0.6)
-		(drill 0.3)
-		(layers "F.Cu" "B.Cu")
-		(net "VDD")
-	)
-	(via
 		(at 127 104)
 		(size 0.6)
@@
 		(net "VDD")
 	)
-	(via
-		(at 139 87.5)
-		(size 0.6)
-		(drill 0.3)
-		(layers "F.Cu" "B.Cu")
-		(net "VDD")
+	(segment
+		(start 134.0425 89.5)
+		(end 135.2 89.5)
+		(width 0.4)
+		(layer "F.Cu")
+		(net "Net-(U2-RFout)")
 	)
 	(segment
-		(start 132.1825 90)
-		(end 132.1825 90.5)
-		(width 0.2)
+		(start 139.732158 88.5)
+		(end 140.52 88.5)
+		(width 0.45)
 		(layer "F.Cu")
-		(net "GNDREF")
+		(net "Net-(U2-RFout)")
 	)
 	(segment
-		(start 144 89.5)
-		(end 143 88.5)
+		(start 135.2 89.5)
+		(end 135.203579 89.503579)
 		(width 0.45)
 		(layer "F.Cu")
-		(net "GNDREF")
+		(net "Net-(U2-RFout)")
 	)
 	(segment
-		(start 151.5 80.43)
-		(end 149.92 80.43)
+		(start 137.187395 89.503579)
+		(end 138.728579 89.503579)
+		(width 0.45)
+		(layer "F.Cu")
+		(net "Net-(U2-RFout)")
+	)
+	(segment
+		(start 135.203579 89.503579)
+		(end 136.5425 89.503579)
+		(width 0.45)
+		(layer "F.Cu")
+		(net "Net-(U2-RFout)")
+	)
+	(segment
+		(start 136.5425 89.503579)
+		(end 137.187395 89.503579)
+		(width 0.45)
+		(layer "F.Cu")
+		(net "Net-(U2-RFout)")
+	)
+	(segment
+		(start 138.728579 89.503579)
+		(end 139.732158 88.5)
+		(width 0.45)
+		(layer "F.Cu")
+		(net "Net-(U2-RFout)")
+	)
+	(segment
+		(start 144.45 92.125)
+		(end 144.5 92.175)
+		(width 0.45)
+		(layer "F.Cu")
+		(net "Net-(F1-B3UL)")
+	)
+	(segment
+		(start 144.45 90.5)
+		(end 144.5 90.45)
+		(width 0.2)
+		(layer "F.Cu")
+		(net "Net-(F1-B3UL)")
+	)
+	(segment
+		(start 144.45 90.5)
+		(end 144.45 92.125)
 		(width 0.45)
 		(layer "F.Cu")
+		(net "Net-(F1-B3UL)")
+	)
+	(segment
+		(start 132.1825 90)
+		(end 132.1825 90.5)
+		(width 0.2)
+		(layer "F.Cu")
 		(net "GNDREF")
 	)
 	(segment
-		(start 141.275 87)
-		(end 142 87)
+		(start 151.5 80.43)
+		(end 149.92 80.43)
 		(width 0.45)
 		(layer "F.Cu")
@@
 	)
 	(segment
+		(start 143 89.5)
+		(end 144.5 89.5)
+		(width 0.45)
+		(layer "F.Cu")
+		(net "GNDREF")
+	)
+	(segment
 		(start 134.0625 86)
 		(end 133.7675 86.295)
@@
 	)
 	(segment
-		(start 144 85.35)
-		(end 143.35 85.35)
-		(width 0.45)
-		(layer "F.Cu")
-		(net "GNDREF")
-	)
-	(segment
 		(start 131 99)
 		(end 131 99.5)
@@
 	)
 	(segment
+		(start 144.5 93.825)
+		(end 144.5 94)
+		(width 0.45)
+		(layer "F.Cu")
+		(net "GNDREF")
+	)
+	(segment
 		(start 112.08 80.43)
 		(end 113.07 80.43)
@@
 	)
 	(segment
-		(start 144.5 89.5)
-		(end 144 89.5)
+		(start 144.5 94)
+		(end 145.5 95)
 		(width 0.45)
 		(layer "F.Cu")
@@
 	)
 	(segment
-		(start 143.35 85.35)
-		(end 143 85)
-		(width 0.45)
-		(layer "F.Cu")
-		(net "GNDREF")
-	)
-	(segment
 		(start 113.07 80.43)
 		(end 113.5 80)
@@
 	)
 	(via
-		(at 143 88.5)
+		(at 143 89.5)
 		(size 0.6)
 		(drill 0.3)
@@
 	)
 	(via
-		(at 144.5 92)
+		(at 145.5 95)
 		(size 0.6)
 		(drill 0.3)
@@
 	)
 	(via
+		(at 139 87.5)
+		(size 0.6)
+		(drill 0.3)
+		(layers "F.Cu" "B.Cu")
+		(net "GNDREF")
+	)
+	(via
 		(at 148 88)
 		(size 0.6)
@@
 	)
 	(via
-		(at 127.5 91)
+		(at 141 86.5)
 		(size 0.6)
 		(drill 0.3)
@@
 	)
 	(via
-		(at 158 85.5)
+		(at 127.5 91)
 		(size 0.6)
 		(drill 0.3)
@@
 	)
 	(via
-		(at 142 87)
+		(at 158 85.5)
 		(size 0.6)
 		(drill 0.3)
@@
 	)
 	(via
-		(at 143 85)
+		(at 143 86.5)
 		(size 0.6)
 		(drill 0.3)
@@
 	)
 	(segment
-		(start 134.0425 89.5)
-		(end 135.2 89.5)
-		(width 0.4)
-		(layer "F.Cu")
-		(net "Net-(U2-RFout)")
-	)
-	(segment
-		(start 139.3625 90.1375)
-		(end 139.725 90.5)
-		(width 0.45)
-		(layer "F.Cu")
-		(net "Net-(U2-RFout)")
-	)
-	(segment
-		(start 135.2 89.5)
-		(end 135.203579 89.503579)
-		(width 0.45)
-		(layer "F.Cu")
-		(net "Net-(U2-RFout)")
-	)
-	(segment
-		(start 139.721421 90.503579)
-		(end 139.725 90.5)
-		(width 0.45)
-		(layer "F.Cu")
-		(net "Net-(U2-RFout)")
-	)
-	(segment
-		(start 137.187395 89.503579)
-		(end 138.728579 89.503579)
-		(width 0.45)
-		(layer "F.Cu")
-		(net "Net-(U2-RFout)")
-	)
-	(segment
-		(start 135.203579 89.503579)
-		(end 136.5425 89.503579)
-		(width 0.45)
-		(layer "F.Cu")
-		(net "Net-(U2-RFout)")
-	)
-	(segment
-		(start 139.725 90.5)
-		(end 140.02 90.5)
-		(width 0.45)
-		(layer "F.Cu")
-		(net "Net-(U2-RFout)")
-	)
-	(segment
-		(start 136.5425 89.503579)
-		(end 137.187395 89.503579)
-		(width 0.45)
-		(layer "F.Cu")
-		(net "Net-(U2-RFout)")
-	)
-	(segment
-		(start 138.728579 89.503579)
-		(end 139.3625 90.1375)
-		(width 0.45)
-		(layer "F.Cu")
-		(net "Net-(U2-RFout)")
-	)
-	(segment
 		(start 132.1825 89.5)
 		(end 129.48 89.5)
@@
 	)
 	(segment
-		(start 144.5 87.5)
-		(end 144 87)
-		(width 0.45)
+		(start 141.53 88.55)
+		(end 141.48 88.5)
+		(width 0.2)
 		(layer "F.Cu")
 		(net "Net-(F1-B3DL)")
@@
 	(segment
 		(start 144.5 88.55)
-		(end 144.5 87.5)
+		(end 144.45 88.5)
 		(width 0.45)
 		(layer "F.Cu")
@@
 	)
 	(segment
-		(start 141.275 90.5)
-		(end 144.45 90.5)
+		(start 144.45 88.5)
+		(end 141.58 88.5)
 		(width 0.45)
 		(layer "F.Cu")
-		(net "Net-(F1-B3UL)")
+		(net "Net-(F1-B3DL)")
 	)
 	(segment
-		(start 144.45 90.5)
-		(end 144.5 90.45)
-		(width 0.2)
+		(start 141.58 88.5)
+		(end 141.53 88.55)
+		(width 0.45)
 		(layer "F.Cu")
-		(net "Net-(F1-B3UL)")
+		(net "Net-(F1-B3DL)")
 	)
 	(segment
