File: pa_usrp_ui.kicad_sch (KiCad schematic)
At the start: 18 parts, among them J1 BWSMA-KE-P001, J2 BWSMA-KE-P001, J3 2118722-2, U1 QPA9418TR13

Commit message: Adding lna uplink
Parts:
- removed C10, C3, C9: 0.1uF, Capacitor_SMD:C_0603_1608Metric, symbol Device:C_US
- removed C2, C6: 10.0uF, Diode_SMD:D_0603_1608Metric, symbol Device:C_Polarized_US
- removed C4, C7: 1000pF, Capacitor_SMD:C_0603_1608Metric, symbol Device:C_US
- removed C8: 100pF, Capacitor_SMD:C_0603_1608Metric, symbol Device:C_US
- removed R1: 0, Resistor_SMD:R_0603_1608Metric, symbol Device:R_US
- removed U1: QPA9418TR13, fooptrints:DFN-14_L7.0-W7.0-P1.06-TL-EP_QPA9418TR13, symbol pa_ui:QPA9418TR13
- added C1, C11, C12, C5: 100pF, Capacitor_SMD:C_0603_1608Metric, symbol Device:C
- added J4: Conn_01x03_Pin, Connector_PinHeader_2.54mm:PinHeader_1x03_P2.54mm_Vertical, symbol Connector:Conn_01x03_Pin
- added J5: HX DC002-1.3, fooptrints:DC-IN-TH_HANXIA_HX-DC002-1.3, symbol Connector:Barrel_Jack_Switch
- added L1: 18nH, Inductor_SMD:L_0603_1608Metric, symbol Device:L
- added R3: 10k, Resistor_SMD:R_0603_1608Metric, symbol Device:R_US
- added R4: 33k, Resistor_SMD:R_0603_1608Metric, symbol Device:R_US
- added U2: TQP3M9036, fooptrints:DFN-8_L2.0-W2.0-P0.50-BL-EP, symbol pa_ui:TQP3M9036
- TP1: value VCC1 -> GND
- TP2: value VCC2 -> SHDIN
Connections:
- net VCC2 is gone; now on net GNDREF: TP1.1
- net GNDREF: now also C11.2, C12.2, J4.1 (Pin_1), J5.2, J5.3, R3.2, U2.1 (NC), U2.3 (NC), U2.4 (NC), U2.5 (NC), U2.8 (NC), U2.9 (EP)
- net at F1.1 (B3DL): now also R2.2
- net at F1.3 (B3UL): now also C5.2; no longer R2.2
- net at J1.5: now also C1.1
- net VCC1 renamed SHDIN
- net SHDIN: now also J4.2 (Pin_2), R4.2
- net VREF renamed VDD
- net VDD: now also C11.1, C12.1, J4.3 (Pin_3), J5.1, L1.1
- new net: R3.1, R4.1, U2.6 (Shutdown)
- new net: C5.1, L1.2, U2.7 (RFout)
- new net: C1.2, U2.2 (RFin)
- no-connect marks 1 -> 0
Other:
- moved on the sheet: TP3

Commit message: adding ngwe
Parts:
- removed C1, C11, C5: 100pF, Capacitor_SMD:C_0603_1608Metric, symbol Device:C
- added C13, C14, C15: 100pF, Capacitor_SMD:C_0402_1005Metric, symbol Device:C
- C12: value 100pF -> 1uF; footprint Capacitor_SMD:C_0603_1608Metric -> Capacitor_SMD:C_0402_1005Metric; lcsc_id (none) -> C52923; price (none) -> 0.0068
- L1: value 18nH -> 68nH; lcsc_id (none) -> C6364697; price (none) -> 0.0414
- R2: price 0.0285 -> 0.0263
- R3: lcsc_id (none) -> C25804; price (none) -> 0.0054
- R4: lcsc_id (none) -> C4216; price (none) -> 0.0021
- U2: price (none) -> 3.1317
Connections:
- net GNDREF: now also C13.2
- net VDD: now also C13.1
- net at L1.2, U2.7 (RFout): now also C14.1
- net at F1.3 (B3UL): now also C14.2
- net at J1.5: now also C15.1
- net at U2.2 (RFin): now also C15.2
Other:
- company: (none) -> UI - Prasimax
- title: (none) -> Low Noise Amplifier
- moved on the sheet: C12, F1, J1, J2, J3, J4, J5, L1, R2, R3, R4, TP1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

Commit message: add lna downlink
Connections:
- net at C14.2: now also F1.1 (B3DL); no longer F1.3 (B3UL)
- net at R2.2: now also F1.3 (B3UL); no longer F1.1 (B3DL)
Changed lines of the file:
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@@
-	(wire
-		(pts
-			(xy 119.38 35.56) (xy 119.38 48.26)
-		)
-		(stroke
-			(width 0)
-			(type default)
-		)
-	)
 	(wire
 		(pts
@@
 	(wire
 		(pts
-			(xy 119.38 48.26) (xy 127 48.26)
-		)
-		(stroke
-			(width 0)
-			(type default)
-		)
-	)
-	(wire
-		(pts
 			(xy 138.43 95.25) (xy 140.97 95.25)
 		)
@@
 	(wire
 		(pts
-			(xy 127 53.34) (xy 110.49 53.34)
-		)
-		(stroke
-			(width 0)
-			(type default)
-		)
-	)
-	(wire
-		(pts
 			(xy 124.46 55.88) (xy 124.46 58.42)
 		)
@@
 	(wire
 		(pts
+			(xy 119.38 35.56) (xy 119.38 53.34)
+		)
+		(stroke
+			(width 0)
+			(type default)
+		)
+	)
+	(wire
+		(pts
 			(xy 124.46 58.42) (xy 124.46 63.5)
 		)
@@
 	(wire
 		(pts
+			(xy 127 53.34) (xy 119.38 53.34)
+		)
+		(stroke
+			(width 0)
+			(type default)
+		)
+	)
+	(wire
+		(pts
 			(xy 48.26 40.64) (xy 45.72 40.64)
 		)
@@
 	(wire
 		(pts
+			(xy 110.49 48.26) (xy 127 48.26)
+		)
+		(stroke
+			(width 0)
+			(type default)
+		)
+	)
+	(wire
+		(pts
 			(xy 53.34 80.01) (xy 53.34 81.28)
 		)
@@
 	(wire
 		(pts
+			(xy 110.49 48.26) (xy 110.49 66.04)
+		)
+		(stroke
+			(width 0)
+			(type default)
+		)
+	)
+	(wire
+		(pts
 			(xy 123.19 95.25) (xy 123.19 90.17)
 		)
@@
 		)
 		(stroke
-			(width 0)
-			(type default)
-		)
-	)
-	(wire
-		(pts
-			(xy 110.49 53.34) (xy 110.49 66.04)
-		)
-		(stroke
